File: KiCAD/PowerSupply.sch (KiCad schematic (older format))
At the start: 0 parts

Commit message: Place power supply from SAMD21-Dev-Board
Parts:
- added C? (x2): 10uF, Capacitors_SMD:C_1206, symbol CP1_Small
- added C?: .1uF, Capacitors_SMD:C_1206, symbol C_Small
- added C? (x2): 2.2uF, Capacitors_SMD:C_1210, symbol C_Small
- added C?: 1.0uF, Capacitors_SMD:C_1210, symbol C_Small
- added F?: 500mA, Resistors_SMD:R_1210, symbol 500mA
- added J?: USB-Micro, 10118192-0001LF:10118192-0001LF, symbol USBAB
- added Q?: 3.7A, 30V, TO_SOT_Packages_SMD:SOT-23, symbol Q_PMOS_GSD
- added R?: 10k, Resistors_SMD:R_1210, symbol R
- added U?: AP2112K-3.3, TO_SOT_Packages_SMD:SOT-23-5, symbol AP2112K-3.3
- added U?: LM1117, symbol LM1117
Connections:
- net labels added: +3.3V, +5V, GND, USB_D+, USB_D-, VBUS, VIN
- wire segments 0 -> 41
- no-connect marks 0 -> 1
Other:
- note added: "If VIN is present, MOSFET will not conduct\nif VIN not present, USB_VBUS will flow through Q1"
- note added: "VIN: 7-15V"

Commit message: Added CAN Bus Sheet
Parts:
- removed J?: USB-Micro, 10118192-0001LF:10118192-0001LF, symbol USBAB
Connections:
- net labels added: +BATT, USB_VBUS, VBAT+, VBAT-
- net labels removed: USB_D+, USB_D-, VBUS, VIN
- wire segments 41 -> 36
- no-connect marks 1 -> 0
Other:
- note added: "0"
- note added: "2/8/19"
- note added: "Author: Matthew Cox\nOrganization: University of Connecticut Formula SAE"
- note added: "Pressure Scanner Board - Power Supply"
- moved on the sheet: C?, F?, Q?, R?, U?

Commit message: Schematic Rev 0
Parts:
- added J2: USB_Micro_B, symbol USB_Micro_B
- added J3: Binder 709 Female Panel Mount, symbol Conn_01x04
- gave numbers to parts that had none: 11
Connections:
- net +BATT: now also J3.3 (Pin_3)
- net GND: now also J2.5 (Pin_5), J3.4 (Pin_4)
- net USB_VBUS: no longer names the net of F1.2
- net USB_VBUS: now also J2.1 (VBUS)
- new net CANH: J3.1 (Pin_1)
- new net CANL: J3.2 (Pin_2)
- new net USB_D+: J2.3 (Pin_3)
- new net USB_D-: J2.2 (Pin_2)
- no-connect marks 0 -> 1
Other:
- note added: "Binder Series 709 Female \nPanel Mount Connector"
- note removed: "If VIN is present, MOSFET will not conduct\nif VIN not present, USB_VBUS will flow through Q1"
- moved on the sheet: C10, C11, C12, C13, C14, C9, F1, Q1, R5, U2, U3

Commit message: Added footprints for all components and created BOM
Parts:
- J2: footprint (none) -> 10104110-0001LF:10104110-0001LF
- J3: footprint (none) -> Pin_Headers:Pin_Header_Straight_1x04_Pitch2.54mm
- U3: footprint (none) -> TO_SOT_Packages_SMD:SOT-223-3_TabPin2
Changed lines of the file:
@@
 $EndDescr
 $Comp
-L GND #PWR022
+L GND #PWR020
 U 1 1 5C631B54
 P 5925 5100
-F 0 "#PWR022" H 5925 4850 50  0001 C CNN
+F 0 "#PWR020" H 5925 4850 50  0001 C CNN
 F 1 "GND" H 5925 4950 50  0000 C CNN
 F 2 "" H 5925 5100 50  0001 C CNN
@@
 $EndComp
 $Comp
-L +5V #PWR023
+L +5V #PWR021
 U 1 1 5C631B6F
 P 6575 4600
-F 0 "#PWR023" H 6575 4450 50  0001 C CNN
+F 0 "#PWR021" H 6575 4450 50  0001 C CNN
 F 1 "+5V" H 6575 4740 50  0000 C CNN
 F 2 "" H 6575 4600 50  0001 C CNN
@@
 $EndComp
 $Comp
-L GND #PWR024
+L GND #PWR022
 U 1 1 5C6327C9
 P 5500 2600
-F 0 "#PWR024" H 5500 2350 50  0001 C CNN
+F 0 "#PWR022" H 5500 2350 50  0001 C CNN
 F 1 "GND" H 5500 2450 50  0000 C CNN
 F 2 "" H 5500 2600 50  0001 C CNN
@@
 $EndComp
 $Comp
-L GND #PWR025
+L GND #PWR023
 U 1 1 5C6327E5
 P 6750 3600
-F 0 "#PWR025" H 6750 3350 50  0001 C CNN
+F 0 "#PWR023" H 6750 3350 50  0001 C CNN
 F 1 "GND" H 6750 3450 50  0000 C CNN
 F 2 "" H 6750 3600 50  0001 C CNN
@@
 $EndComp
 $Comp
-L +3.3V #PWR026
+L +3.3V #PWR024
 U 1 1 5C6327F2
 P 7400 2900
-F 0 "#PWR026" H 7400 2750 50  0001 C CNN
+F 0 "#PWR024" H 7400 2750 50  0001 C CNN
 F 1 "+3.3V" H 7400 3040 50  0000 C CNN
 F 2 "" H 7400 2900 50  0001 C CNN
@@
 $EndComp
 $Comp
-L GND #PWR027
+L GND #PWR025
 U 1 1 5C6327FF
 P 5450 3500
-F 0 "#PWR027" H 5450 3250 50  0001 C CNN
+F 0 "#PWR025" H 5450 3250 50  0001 C CNN
 F 1 "GND" H 5450 3350 50  0000 C CNN
 F 2 "" H 5450 3500 50  0001 C CNN
@@
 $EndComp
 $Comp
-L +5V #PWR028
+L +5V #PWR026
 U 1 1 5C632805
 P 6300 2850
-F 0 "#PWR028" H 6300 2700 50  0001 C CNN
+F 0 "#PWR026" H 6300 2700 50  0001 C CNN
 F 1 "+5V" H 6300 2990 50  0000 C CNN
 F 2 "" H 6300 2850 50  0001 C CNN
@@
 $EndComp
 $Comp
-L GND #PWR029
+L GND #PWR027
 U 1 1 5C63283C
 P 5325 4950
-F 0 "#PWR029" H 5325 4700 50  0001 C CNN
+F 0 "#PWR027" H 5325 4700 50  0001 C CNN
 F 1 "GND" H 5325 4800 50  0000 C CNN
 F 2 "" H 5325 4950 50  0001 C CNN
@@
 F 0 "U3" H 5775 4825 50  0000 C CNN
 F 1 "LM1117" H 5925 4825 50  0000 L CNN
-F 2 "" H 5925 4700 50  0001 C CNN
+F 2 "TO_SOT_Packages_SMD:SOT-223-3_TabPin2" H 5925 4700 50  0001 C CNN
 F 3 "" H 5925 4700 50  0001 C CNN
 	1    5925 4700
@@
 $EndComp
 $Comp
-L +5V #PWR030
+L +5V #PWR028
 U 1 1 5C633AAC
 P 5500 2125
-F 0 "#PWR030" H 5500 1975 50  0001 C CNN
+F 0 "#PWR028" H 5500 1975 50  0001 C CNN
 F 1 "+5V" H 5500 2265 50  0000 C CNN
 F 2 "" H 5500 2125 50  0001 C CNN
@@
 0
 $Comp
-L +BATT #PWR031
+L +BATT #PWR029
 U 1 1 5C64B882
 P 5325 4600
-F 0 "#PWR031" H 5325 4450 50  0001 C CNN
+F 0 "#PWR029" H 5325 4450 50  0001 C CNN
 F 1 "+BATT" H 5325 4740 50  0000 C CNN
 F 2 "" H 5325 4600 50  0001 C CNN
@@
 F 0 "J3" H 4500 4800 50  0000 C CNN
 F 1 "Binder 709 Female Panel Mount" H 4500 4300 50  0001 C CNN
-F 2 "" H 4500 4600 50  0001 C CNN
+F 2 "Pin_Headers:Pin_Header_Straight_1x04_Pitch2.54mm" H 4500 4600 50  0001 C CNN
 F 3 "" H 4500 4600 50  0001 C CNN
 	1    4500 4600
@@
 F 0 "J2" H 4200 3500 50  0000 C CNN
 F 1 "USB_Micro_B" H 4210 2895 50  0000 C CNN
-F 2 "" H 4200 3200 50  0001 C CNN
+F 2 "10104110-0001LF:10104110-0001LF" H 4200 3200 50  0001 C CNN
 F 3 "" H 4200 3200 50  0001 C CNN
 	1    4200 3200
@@
 NoConn ~ 4400 3300
 $Comp
-L GND #PWR032
+L GND #PWR030
 U 1 1 5C661C2D
 P 4700 3550
-F 0 "#PWR032" H 4700 3300 50  0001 C CNN
+F 0 "#PWR030" H 4700 3300 50  0001 C CNN
 F 1 "GND" H 4700 3400 50  0000 C CNN
 F 2 "" H 4700 3550 50  0001 C CNN

Commit message: More layout
Connections:
- net VBUS: now reaches F1.2, J2.1 (VBUS)
Changed lines of the file:
@@
+	1    0    0    -1
+$EndComp
+$Comp
+L VBUS #PWR?
+U 1 1 5C938C3A
+P 4675 2900
+F 0 "#PWR?" H 4675 2750 50  0001 C CNN
+F 1 "VBUS" H 4675 3050 50  0000 C CNN
+F 2 "" H 4675 2900 50  0001 C CNN
+F 3 "" H 4675 2900 50  0001 C CNN
+	1    4675 2900
 	1    0    0    -1
 $EndComp
@@
 Wire Wire Line
 	5325 4800 4700 4800
+Wire Wire Line
+	4675 2900 4675 3000
+Connection ~ 4675 3000
 $EndSCHEMATC
