File: KiCAD/CAN-BUS.sch (KiCad schematic (older format))
At the start: 11 parts, among them U13 MCP2551, U14 MCP2515, Y2 16MHz

Commit message: Finished layout V0.01
Connections:
- net CANH+ renamed CAN+
- net CANL- renamed CAN-
Other:
- note added: "Named this way so pcbnew\nacknowledges differential pair\n"
Changed lines of the file:
@@
 OSC-
 Text GLabel 9600 3700 2    39   Input ~ 0
-CANH+
+CAN+
 Text GLabel 9600 3800 2    39   Input ~ 0
-CANL-
+CAN-
 NoConn ~ 4750 4025
+Text Notes 9600 4050 0    39   ~ 0
+Named this way so pcbnew\nacknowledges differential pair\n
 $EndSCHEMATC
